Commit message: Created simulation model

File: description/gazebo_control_diff.xacro (robot description, xacro)
@@ -6,5 +6,5 @@
             <left_joint>left_wheel_joint</left_joint>
             <right_joint>right_wheel_joint</right_joint>
-            <wheel_separation>0.08</wheel_separation>
+            <wheel_separation>0.1</wheel_separation>
             <wheel_diameter>0.06</wheel_diameter>
             <!-- Limits -->
@@ -18,4 +18,7 @@
             <publish_wheel_tf>true</publish_wheel_tf>
         </plugin>
+        <plugin name="gazebo_ros2_control" filename="libgazebo_ros2_control.so">
+            <parameters>$(find my_bot)/config/my_controllers.yaml</parameters>
+        </plugin>
     </gazebo>
 </robot>

File: description/robot_core.xacro (robot description, xacro)
@@ -45,8 +45,8 @@
     </gazebo>
     <!-- LEFT WHEEL LINK -->
-    <joint name="left_wheel_joint" type="continuous">
-        <parent link="base_link"/>
+    <!-- <joint name="left_wheel_joint" type="continuous">
+        <parent link="chassis"/>
         <child link="left_wheel"/>
-        <origin xyz="0 0.05 0.01" rpy="-${pi/2} 0 0"/>
+        <origin xyz="0.04 0.05 0.01" rpy="-${pi/2} 0 0"/>
         <axis xyz="0 0 1"/>
     </joint>
@@ -69,10 +69,10 @@
     <gazebo reference="left_wheel">
         <material>Gazebo/Blue</material>
-    </gazebo>
+    </gazebo> -->
     <!-- RIGHT WHEEL LINK -->
-    <joint name="right_wheel_joint" type="continuous">
-        <parent link="base_link"/>
+    <!-- <joint name="right_wheel_joint" type="continuous">
+        <parent link="chassis"/>
         <child link="right_wheel"/>
-        <origin xyz="0 -0.05 0.01" rpy="${pi/2} 0 0"/>
+        <origin xyz="0.04 -0.05 0.01" rpy="${pi/2} 0 0"/>
         <axis xyz="0 0 -1"/>
     </joint>
@@ -95,10 +95,10 @@
     <gazebo reference="right_wheel">
         <material>Gazebo/Blue</material>
-    </gazebo>
+    </gazebo> -->
     <!-- FRONT CASTER WHEEL -->
-    <joint name="caster_wheel_front_joint" type="fixed">
+    <!-- <joint name="caster_wheel_front_joint" type="fixed">
         <parent link="chassis"/>
         <child link="caster_wheel_front"/>
-        <origin xyz="0.18 0 0.011" rpy="0 0 0"/>
+        <origin xyz="0.15 0 0.011" rpy="0 0 0"/>
     </joint>
     <link name="caster_wheel_front">
@@ -118,7 +118,9 @@
     <gazebo reference="caster_wheel_front">
         <material>Gazebo/Black</material>
-    </gazebo>
+        <mu1 value="0.0001"/>
+        <mu2 value="0.0001"/>
+    </gazebo> -->
     <!-- REAR CASTER WHEEL -->
-    <joint name="caster_wheel_rear_joint" type="fixed">
+    <!-- <joint name="caster_wheel_rear_joint" type="fixed">
         <parent link="chassis"/>
         <child link="caster_wheel_rear"/>
@@ -141,4 +143,4 @@
     <gazebo reference="caster_wheel_rear">
         <material>Gazebo/Black</material>
-    </gazebo>
+    </gazebo> -->
 </robot>

Commit message: update

File: description/gazebo_control_diff.xacro (robot description, xacro)
@@ -4,6 +4,6 @@
         <plugin name='diff_drive' filename='libgazebo_ros_diff_drive.so'>
             <!-- Wheel Information -->
-            <left_joint>left_wheel_joint</left_joint>
-            <right_joint>right_wheel_joint</right_joint>
+            <left_joint>rear_left_wheel_joint</left_joint>
+            <right_joint>front_right_wheel_joint</right_joint>
             <wheel_separation>0.1</wheel_separation>
             <wheel_diameter>0.06</wheel_diameter>
@@ -18,7 +18,4 @@
             <publish_wheel_tf>true</publish_wheel_tf>
         </plugin>
-        <plugin name="gazebo_ros2_control" filename="libgazebo_ros2_control.so">
-            <parameters>$(find my_bot)/config/my_controllers.yaml</parameters>
-        </plugin>
     </gazebo>
 </robot>

File: description/robot.urdf.xacro (robot description, xacro)
@@ -1,6 +1,8 @@
 <?xml version="1.0"?>
 <robot xmlns:xacro="http://www.ros.org/wiki/xacro"  name="robot">
-    <xacro:include filename="robot_core.xacro" />
+    <xacro:include filename="robot_core_diff.xacro" />
     <!-- <xacro:include filename="gazebo_control_diff.xacro" /> -->
     <xacro:include filename="ros2_control.xacro" />
+    <xacro:include filename="camera.xacro" />
+    <!-- <xacro:include filename="lidar.xacro" /> -->
 </robot>

File: description/robot_core_diff.xacro (robot description, xacro)
@@ -47,12 +47,12 @@
         <material>Gazebo/White</material>
     </gazebo>
-    <!-- REAR LEFT WHEEL LINK -->
-    <joint name="rear_left_wheel_joint" type="continuous">
+    <!-- LEFT WHEEL LINK -->
+    <joint name="left_wheel_joint" type="continuous">
         <parent link="chassis"/>
-        <child link="rear_left_wheel"/>
+        <child link="left_wheel"/>
         <origin xyz="0.04 0.05 0.01" rpy="-${pi/2} 0 0"/>
         <axis xyz="0 0 1"/>
     </joint>
-    <link name="rear_left_wheel">
+    <link name="left_wheel">
         <visual>
             <geometry>
@@ -70,15 +70,15 @@
         </xacro:inertial_cylinder>
     </link>
-    <gazebo reference="rear_left_wheel">
+    <gazebo reference="left_wheel">
         <material>Gazebo/Blue</material>
     </gazebo>
-    <!-- FRONT LEFT WHEEL LINK -->
-    <joint name="front_left_wheel_joint" type="continuous">
+    <!-- REAR RIGHT WHEEL LINK -->
+    <joint name="right_wheel_joint" type="continuous">
         <parent link="chassis"/>
-        <child link="front_left_wheel"/>
-        <origin xyz="0.14 0.05 0.01" rpy="-${pi/2} 0 0"/>
-        <axis xyz="0 0 1"/>
+        <child link="right_wheel"/>
+        <origin xyz="0.04 -0.05 0.01" rpy="${pi/2} 0 0"/>
+        <axis xyz="0 0 -1"/>
     </joint>
-    <link name="front_left_wheel">
+    <link name="right_wheel">
         <visual>
             <geometry>
@@ -96,61 +96,9 @@
         </xacro:inertial_cylinder>
     </link>
-    <gazebo reference="front_left_wheel">
-        <material>Gazebo/Blue</material>
-    </gazebo>
-    <!-- REAR RIGHT WHEEL LINK -->
-    <joint name="rear_right_wheel_joint" type="continuous">
-        <parent link="chassis"/>
-        <child link="rear_right_wheel"/>
-        <origin xyz="0.04 -0.05 0.01" rpy="${pi/2} 0 0"/>
-        <axis xyz="0 0 -1"/>
-    </joint>
-    <link name="rear_right_wheel">
-        <visual>
-            <geometry>
-                <cylinder radius="0.03" length="0.025"/>
-            </geometry>
-            <material name="blue"/>
-        </visual>
-        <collision>
-            <geometry>
-                <cylinder radius="0.03" length="0.025"/>
-            </geometry>
-        </collision>
-        <xacro:inertial_cylinder mass="0.01" length="0.025" radius="0.03">
-            <origin xyz="0 0 0" rpy="0 0 0"/>
-        </xacro:inertial_cylinder>
-    </link>
-    <gazebo reference="rear_right_wheel">
-        <material>Gazebo/Blue</material>
-    </gazebo>
-    <!-- FRONT RIGHT WHEEL LINK -->
-    <joint name="front_right_wheel_joint" type="continuous">
-        <parent link="chassis"/>
-        <child link="front_right_wheel"/>
-        <origin xyz="0.14 -0.05 0.01" rpy="${pi/2} 0 0"/>
-        <axis xyz="0 0 -1"/>
-    </joint>
-    <link name="front_right_wheel">
-        <visual>
-            <geometry>
-                <cylinder radius="0.03" length="0.025"/>
-            </geometry>
-            <material name="blue"/>
-        </visual>
-        <collision>
-            <geometry>
-                <cylinder radius="0.03" length="0.025"/>
-            </geometry>
-        </collision>
-        <xacro:inertial_cylinder mass="0.01" length="0.025" radius="0.03">
-            <origin xyz="0 0 0" rpy="0 0 0"/>
-        </xacro:inertial_cylinder>
-    </link>
-    <gazebo reference="front_right_wheel">
+    <gazebo reference="right_wheel">
         <material>Gazebo/Blue</material>
     </gazebo>
     <!-- FRONT CASTER WHEEL -->
-    <!-- <joint name="caster_wheel_front_joint" type="fixed">
+    <joint name="caster_wheel_front_joint" type="fixed">
         <parent link="chassis"/>
         <child link="caster_wheel_front"/>
@@ -173,7 +121,7 @@
     <gazebo reference="caster_wheel_front">
         <material>Gazebo/Black</material>
-        <mu1 value="0..1"/>
-        <mu1 value="0..1"/>
-    </gazebo> -->
+        <mu1 value="0.001"/>
+        <mu2 value="0.001"/>
+    </gazebo>
     <!-- REAR CASTER WHEEL -->
     <!-- <joint name="caster_wheel_rear_joint" type="fixed">
